File: electronic/robot_main_board/robot_main_board.brd (EAGLE design)
At the start: 100 x 123.2 mm, 28 parts, among them J1 HORIZONTAL_ROTATE, J10 joint2_ends_min, J11 joint2_ends_max, J13 hr_ends_max, J2 JOINT_1, J3 JOINT_2, J4 JOYSTICK, J5 joint1_en_sw, J6 joint2_en_sw, J7 hr_en_sw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

Commit message: change robot_main_board
Parts:
- added J20: power, SparkFun-Connectors:MOLEX-1X2
Connections:
- net GND: now also J20.1
- net V+: now also J20.2
Routing:
- net GND: track 101.2 -> 160.6 mm
- net V+: track 6.35 -> 44.4 mm
Changed lines of the file:
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@@
 <layer number="43" name="vRestrict" color="2" fill="10" visible="yes" active="yes"/>
 <layer number="44" name="Drills" color="7" fill="1" visible="no" active="yes"/>
-<layer number="45" name="Holes" color="7" fill="1" visible="no" active="yes"/>
+<layer number="45" name="Holes" color="7" fill="1" visible="yes" active="yes"/>
 <layer number="46" name="Milling" color="3" fill="1" visible="no" active="yes"/>
 <layer number="47" name="Measures" color="7" fill="1" visible="no" active="yes"/>
@@
 <wire x1="0" y1="80" x2="0" y2="-43.18" width="0" layer="20"/>
 <wire x1="7.62" y1="43.18" x2="7.62" y2="29.21" width="1.27" layer="21"/>
+<hole x="95.25" y="76.2" drill="3"/>
+<hole x="3.81" y="76.2" drill="3"/>
+<hole x="3.81" y="-39.37" drill="3"/>
+<hole x="95.25" y="-39.37" drill="3"/>
 </plain>
 <attributes>
@@
 <element name="J18" library="SparkFun-Connectors" package="1X07" value="" x="19.05" y="8.89" rot="R270"/>
 <element name="J19" library="SparkFun-Connectors" package="1X05" value="" x="19.05" y="-22.86" rot="R90"/>
+<element name="J20" library="SparkFun-Connectors" package="MOLEX-1X2" value="power" x="6.35" y="6.35" rot="R90">
+<attribute name="SF_ID" value="PRT-09918" x="6.35" y="6.35" size="1.778" layer="27" rot="R90" display="off"/>
+</element>
 </elements>
 <signals>
@@
 <contactref element="J18" pad="3"/>
 <wire x1="20.32" y1="3.81" x2="19.05" y2="3.81" width="1.27" layer="16"/>
-<wire x1="19.05" y1="3.81" x2="19.05" y2="6.35" width="1.27" layer="16"/>
+<wire x1="19.05" y1="3.81" x2="19.05" y2="5.08" width="1.27" layer="16"/>
+<wire x1="19.05" y1="5.08" x2="19.05" y2="6.35" width="1.27" layer="16"/>
 <wire x1="19.05" y1="6.35" x2="25.4" y2="6.35" width="1.27" layer="16"/>
-<wire x1="83.82" y1="24.13" x2="83.82" y2="31.75" width="0" layer="19" extent="1-1"/>
+<contactref element="J20" pad="1"/>
+<wire x1="6.35" y1="6.35" x2="7.62" y2="6.35" width="1.27" layer="16"/>
+<wire x1="7.62" y1="6.35" x2="8.89" y2="6.35" width="1.27" layer="16"/>
+<wire x1="8.89" y1="6.35" x2="10.16" y2="6.35" width="1.27" layer="16"/>
+<wire x1="10.16" y1="6.35" x2="11.43" y2="6.35" width="1.27" layer="16"/>
+<wire x1="11.43" y1="6.35" x2="12.7" y2="6.35" width="1.27" layer="16"/>
+<wire x1="12.7" y1="6.35" x2="13.97" y2="6.35" width="1.27" layer="16"/>
+<wire x1="13.97" y1="6.35" x2="15.24" y2="6.35" width="1.27" layer="16"/>
+<wire x1="15.24" y1="6.35" x2="16.51" y2="6.35" width="1.27" layer="16"/>
+<wire x1="16.51" y1="6.35" x2="19.05" y2="6.35" width="1.27" layer="16"/>
+<wire x1="8.89" y1="3.81" x2="10.16" y2="3.81" width="1.27" layer="16"/>
+<wire x1="10.16" y1="3.81" x2="11.43" y2="3.81" width="1.27" layer="16"/>
+<wire x1="11.43" y1="3.81" x2="12.7" y2="3.81" width="1.27" layer="16"/>
+<wire x1="12.7" y1="3.81" x2="13.97" y2="3.81" width="1.27" layer="16"/>
+<wire x1="13.97" y1="3.81" x2="15.24" y2="3.81" width="1.27" layer="16"/>
+<wire x1="15.24" y1="3.81" x2="16.51" y2="3.81" width="1.27" layer="16"/>
+<wire x1="16.51" y1="3.81" x2="17.78" y2="3.81" width="1.27" layer="16"/>
+<wire x1="17.78" y1="3.81" x2="19.05" y2="3.81" width="1.27" layer="16"/>
+<wire x1="6.35" y1="6.35" x2="7.62" y2="5.08" width="1.27" layer="16"/>
+<wire x1="7.62" y1="5.08" x2="8.89" y2="3.81" width="1.27" layer="16"/>
+<wire x1="7.62" y1="6.35" x2="7.62" y2="5.08" width="1.27" layer="16"/>
+<wire x1="8.89" y1="6.35" x2="8.89" y2="3.81" width="1.27" layer="16"/>
+<wire x1="10.16" y1="6.35" x2="10.16" y2="3.81" width="1.27" layer="16"/>
+<wire x1="11.43" y1="6.35" x2="11.43" y2="3.81" width="1.27" layer="16"/>
+<wire x1="12.7" y1="6.35" x2="12.7" y2="3.81" width="1.27" layer="16"/>
+<wire x1="13.97" y1="6.35" x2="13.97" y2="3.81" width="1.27" layer="16"/>
+<wire x1="15.24" y1="6.35" x2="15.24" y2="3.81" width="1.27" layer="16"/>
+<wire x1="15.24" y1="6.35" x2="16.51" y2="5.08" width="1.27" layer="16"/>
+<wire x1="16.51" y1="5.08" x2="16.51" y2="3.81" width="1.27" layer="16"/>
+<wire x1="16.51" y1="6.35" x2="17.78" y2="5.08" width="1.27" layer="16"/>
+<wire x1="17.78" y1="5.08" x2="17.78" y2="3.81" width="1.27" layer="16"/>
+<wire x1="17.78" y1="5.08" x2="19.05" y2="5.08" width="1.27" layer="16"/>
+<wire x1="82.2826" y1="25.3981875" x2="83.1831875" y2="24.4976" width="1.27" layer="16"/>
+<wire x1="83.82" y1="31.75" x2="83.82" y2="31.3842125" width="1.27" layer="16"/>
+<wire x1="83.82" y1="31.3842125" x2="82.2826" y2="29.8468125" width="1.27" layer="16"/>
+<wire x1="83.1831875" y1="24.4976" x2="83.4524" y2="24.4976" width="1.27" layer="16"/>
+<wire x1="83.4524" y1="24.4976" x2="83.82" y2="24.13" width="1.27" layer="16"/>
+<wire x1="82.2826" y1="29.8468125" x2="82.2826" y2="25.3981875" width="1.27" layer="16"/>
 </signal>
 <signal name="+5V">
@@
 <contactref element="B1" pad="VIN"/>
 <contactref element="J18" pad="1"/>
-<wire x1="19.05" y1="8.89" x2="25.4" y2="8.89" width="1.27" layer="16"/>
+<wire x1="19.05" y1="8.89" x2="22.86" y2="8.89" width="1.27" layer="16"/>
+<contactref element="J20" pad="2"/>
+<wire x1="22.86" y1="8.89" x2="25.4" y2="8.89" width="1.27" layer="16"/>
+<wire x1="6.35" y1="8.89" x2="19.05" y2="8.89" width="1.27" layer="16"/>
+<wire x1="25.4" y1="10.16" x2="25.4" y2="8.89" width="1.27" layer="16"/>
+<wire x1="6.35" y1="8.89" x2="6.35" y2="10.16" width="1.27" layer="16"/>
+<wire x1="6.35" y1="10.16" x2="25.4" y2="10.16" width="1.27" layer="16"/>
+<wire x1="25.4" y1="10.16" x2="26.67" y2="10.16" width="1.27" layer="16"/>
+<wire x1="26.67" y1="8.89" x2="26.67" y2="10.16" width="1.27" layer="16"/>
+<wire x1="25.4" y1="8.89" x2="26.67" y2="8.89" width="1.27" layer="16"/>
 </signal>
 <signal name="+3V3">
